File: kicad/old_rev/PCB_2/usb2ps1mouse.kicad_sch (KiCad schematic)
At the start: 11 parts, among them J1 Conn_01x09_Pin, J2 USB_A, J3 Conn_01x02, J4 Conn_01x02, U1 RP2040-Zero, U3 AMS1117-5.0

Commit message: Add PCB_3 board revision.
Parts:
- removed J3, J4: Conn_01x02, Jumper:SolderJumper-2_P1.3mm_Open_RoundedPad1.0x1.5mm, symbol Connector_Generic:Conn_01x02
- removed U3: AMS1117-5.0, Package_TO_SOT_SMD:SOT-223-3_TabPin2, symbol Regulator_Linear:AMS1117-5.0
- added D1: SS14, Diode_SMD:D_SMA, symbol Diode:SS14
- added L1: 22u, usb2ps1mouse-specific:L_combo, symbol Device:L
- added U2: ME2108A50PG, Package_TO_SOT_SMD:SOT-89-3, symbol usb2ps1mouse_specific:ME2108A50PG_SOT89-3
Connections:
- net +5V: now also C1.1, U1.23 (5V), D1.1 (K), U2.2 (Vout)
- net GND: now also U2.1 (Vss)
- net VCON: now also L1.1
- net VMOT: no longer names the net of J1.3 (Pin_3)
- net VMOT: no longer C1.1
- new net: D1.2 (A), L1.2, U2.3 (Lx)
- no-connect marks 1 -> 2
Other:
- note added: "DC 3.3V to DC 5V step-up"
- note removed: "7.5V to 5V"
- moved on the sheet: C1, C2
